File: Hardware/Turing_mini_expander.brd (EAGLE design)
At the start: 106 x 19.5 mm, 21 parts, among them U1 TL072_

Commit message: Rev 3 PCB
Reverses order of pots
Connections:
- net GATE1: now also VR6.3; no longer VR2.3
- net GATE2: now also VR5.3; no longer VR3.3
- net GATE4: now also VR3.3; no longer VR5.3
- net GATE5: now also VR2.3; no longer VR6.3
Routing:
- net GATE4: track 94.3 -> 38.1 mm, vias 4 -> 1
- net GATE1: track 36.7 -> 91.6 mm, vias 2 -> 1
- net GATE2: track 37.6 -> 81.8 mm, vias 2 -> 1
- net GATE6: track 71.8 -> 32.3 mm
- net GATE5: track 85.7 -> 54.5 mm, vias 3 -> 2
- net GATE7: track 47.0 -> 31.5 mm, vias 3 -> 1
- net CLOCK: track 45.8 -> 34.3 mm, vias 3 -> 1
- net GATE3: track 59.8 -> 51.2 mm, vias 2 -> 0
- net N$6: track 20.3 -> 28.8 mm, vias 0 -> 1
- net -12V: track 53.6 -> 60.7 mm
- net GND: track 6.33 -> 0.00 mm, vias 3 -> 0
- net +12V: track 59.6 -> 64.6 mm
- net GATE8: track 35.0 -> 31.2 mm, vias 2 -> 1
- net N$2: track 15.7 -> 16.9 mm, vias 0 -> 1
- net N$4: track 11.5 -> 12.3 mm
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Other:
- board text added: "PCB rev 3 June 2016 musicthing.co.uk"
- board text added: "Turing Machine Mini Voltage Expander Designed in Portscatho Cornwall by Tom Whitwell"
- board text removed: "Turing Machine Mini Voltage Expander Designed in Portscatho Cornwall by Tom Whitwell PCB rev 2 September 2015 musicthing.co.uk"
