File: Hardware/Turing_mini_expander.sch (EAGLE design)
At the start: 20 parts, among them U1 TL072_

Commit message: Rev 3 PCB
Reverses order of pots
Connections:
- net GATE1: now also VR6.E; no longer VR2.E
- net GATE2: now also VR5.E; no longer VR3.E
- net GATE4: now also VR3.E; no longer VR5.E
- net GATE5: now also VR2.E; no longer VR6.E
Changed lines of the file:
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@@
 <?xml version="1.0" encoding="utf-8"?>
 <!DOCTYPE eagle SYSTEM "eagle.dtd">
-<eagle version="7.2.0">
+<eagle version="7.4.0">
 <drawing>
 <settings>
@@
 </variantdefs>
 <classes>
-<class number="0" name="default" width="0.254" drill="0">
+<class number="0" name="default" width="0" drill="0">
 </class>
-<class number="1" name="power" width="0.4064" drill="0">
+<class number="1" name="power" width="0" drill="0">
 </class>
-<class number="2" name="ground" width="0.4064" drill="0">
+<class number="2" name="ground" width="0" drill="0">
 </class>
 </classes>
@@
 </segment>
 <segment>
-<pinref part="VR2" gate="G$1" pin="E"/>
-<wire x1="83.82" y1="157.48" x2="43.18" y2="157.48" width="0.1524" layer="91"/>
-<label x="43.18" y="157.48" size="1.778" layer="95" rot="R180" xref="yes"/>
+<pinref part="VR6" gate="G$1" pin="E"/>
+<wire x1="63.5" y1="40.64" x2="83.82" y2="40.64" width="0.1524" layer="91"/>
+<label x="63.5" y="40.64" size="1.778" layer="95" rot="R180" xref="yes"/>
 </segment>
 </net>
@@
 </segment>
 <segment>
-<pinref part="VR3" gate="G$1" pin="E"/>
-<wire x1="83.82" y1="127" x2="43.18" y2="127" width="0.1524" layer="91"/>
-<label x="43.18" y="127" size="1.778" layer="95" rot="R180" xref="yes"/>
+<pinref part="VR5" gate="G$1" pin="E"/>
+<wire x1="63.5" y1="71.12" x2="83.82" y2="71.12" width="0.1524" layer="91"/>
+<label x="63.5" y="71.12" size="1.778" layer="95" rot="R180" xref="yes"/>
 </segment>
 </net>
@@
 <segment>
 <pinref part="VR4" gate="G$1" pin="E"/>
-<wire x1="83.82" y1="99.06" x2="43.18" y2="99.06" width="0.1524" layer="91"/>
-<label x="43.18" y="99.06" size="1.778" layer="95" rot="R180" xref="yes"/>
+<wire x1="63.5" y1="99.06" x2="83.82" y2="99.06" width="0.1524" layer="91"/>
+<label x="63.5" y="99.06" size="1.778" layer="95" rot="R180" xref="yes"/>
 </segment>
 </net>
@@
 </segment>
 <segment>
-<pinref part="VR5" gate="G$1" pin="E"/>
-<wire x1="83.82" y1="71.12" x2="43.18" y2="71.12" width="0.1524" layer="91"/>
-<label x="43.18" y="71.12" size="1.778" layer="95" rot="R180" xref="yes"/>
+<pinref part="VR3" gate="G$1" pin="E"/>
+<wire x1="63.5" y1="127" x2="83.82" y2="127" width="0.1524" layer="91"/>
+<label x="63.5" y="127" size="1.778" layer="95" rot="R180" xref="yes"/>
 </segment>
 </net>
@@
 </segment>
 <segment>
-<pinref part="VR6" gate="G$1" pin="E"/>
-<wire x1="83.82" y1="40.64" x2="43.18" y2="40.64" width="0.1524" layer="91"/>
-<label x="43.18" y="40.64" size="1.778" layer="95" rot="R180" xref="yes"/>
-</segment>
-</net>
+<pinref part="VR2" gate="G$1" pin="E"/>
+<wire x1="66.04" y1="157.48" x2="83.82" y2="157.48" width="0.1524" layer="91"/>
+<label x="63.5" y="157.48" size="1.778" layer="95" rot="R180" xref="yes"/>
+</segment>
+</net>
